File: HANDy.kicad_sch (KiCad schematic)
At the start: 104 parts, among them IC1 INA241A2IDDFR, IC2 INA241A2IDDFR, IC3 INA241A2IDDFR, IC4 INA241A2IDDFR, IC5 INA241A2IDDFR, IC6 INA241A2IDDFR, J1 8000078306, J2 Motor1, J3 Motor2, J4 Motor3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

Commit message: manually fixed component labels in schematic
kicad imported them without their numbers
Parts:
- renumbered R7 to R8
Other:
- title: (none) -> HANDyDriver
